Commit message: Better Clock Synchronization
1- added clock sync with CoppeliaSim and moveit
2-separate 2 node one for moveing the robot and the other sensing the robot position

File: src/abb_irb_sim_v2/urdf/abb_irb_sim_v2.urdf (robot description, URDF)
Before this commit: robot abb_irb_sim_v2, 9 links, 8 joints
Joints:
- joint joint1: limit (none) -> lower=-2.8797932658 upper=2.8797932658 effort=1000 velocity=4.36332313; type continuous -> revolute
- joint joint2: limit (none) -> lower=-1.9198621772 upper=1.9198621772 effort=1000 velocity=4.36332313; type continuous -> revolute
- joint joint3: limit (none) -> lower=-1.9198621772 upper=1.2217304764 effort=1000 velocity=4.36332313; type continuous -> revolute
- joint joint4: limit (none) -> lower=-2.7925268032 upper=2.7925268032 effort=1000 velocity=5.5850536064; type continuous -> revolute
- joint joint5: limit (none) -> lower=-2.0943951024 upper=2.0943951024 effort=1000 velocity=5.5850536064; type continuous -> revolute
- joint joint6: limit (none) -> lower=-6.981317008 upper=6.981317008 effort=1000 velocity=7.3303828584; type continuous -> revolute
